File: hardware/shield/hrm-shield.sch (EAGLE design)
At the start: 37 parts, among them IC3 FM25-DFN, T2 BC846, U1 EM406FLAT, U2 EM406FLAT, U4 EM406FLAT, U5 ADXL362, U6 W25Q16BVZP, U7 MPU-9250, X1 NRF51822-RIGHT

Commit message: scheme with ada1292
Parts:
- removed U1, U2, U4: EM406FLAT, icarus_sensors:EM406FLAT
- removed U5: ADXL362, icarus_sensors:ADXL362ADXL362-1:1
- added C15, C18, C19, C20: 1uF, SparkFun-Capacitors:0.1UF-25V(+80/-20%)(0603)
- added C16, C21: 0.1uF, SparkFun-Capacitors:0.1UF-25V(+80/-20%)(0603)
- added C17: 4.7nF, SparkFun-Capacitors:0.1UF-25V(+80/-20%)(0603)
- added C22: 1.5nF, SparkFun-Capacitors:0.1UF-25V(+80/-20%)(0603)
- added C23, C24, C25, C26: 47pF, SparkFun-Capacitors:0.1UF-25V(+80/-20%)(0603)
- added R10: 1M, SparkFun-Resistors:100OHM1/10W1%(0603)
- added R11, R3: 0, SparkFun-Resistors:100OHM1/10W1%(0603)
- added R12, R8: 100K, SparkFun-Resistors:100OHM1/10W1%(0603)
- added R13, R14, R15, R16: 51K, SparkFun-Resistors:100OHM1/10W1%(0603)
- added U$3: ADS1292, icarus_sensors:ADS1292
- added U$6: EM406-2PINFLAT, icarus_sensors:EM406-2PINFLAT
- C1: value 0.1uF -> 4.7nF
- C3: value 10nF -> 1uF
- C4, C5: value 0.1uF -> 1uF
- U7: value MPU-9250 -> EM406-2PINFLAT; device icarus_sensors:MPU-9250 -> icarus_sensors:EM406-2PINFLAT
Connections:
- removed net ADXL_CS: U$1P0.23.S, U5.!CS
- removed net ADXL_DATA: U$1P0.21.S, U5.INT1
- removed net ADXL_FSYNC: U$1P0.22.S, U5.INT2
- removed net BAR1_CS: U$1P0.25.S, U1.CSB
- removed net BAR2_CS: U4.CSB, X1P0.20.S
- removed net BAR3_CS: U2.CSB, X1P0.19.S
- removed net MPU_CS: U7.NCS, X1P0.18.S
- removed net MPU_FSYNC: U7.FSYNC, X1P0.17.S
- removed net VCCIO: C6.1, U5.VDDIO
- new net ADS_CLK: U$1P0.25.S, U$3.CLK
- new net ADS_CLKSEL: U$1P0.22.S, U$3.CLKSEL
- new net ADS_CS: U$1P0.23.S
- new net ADS_DATA: U$1P0.21.S, U$3.DRDY
- new net ADS_GPIO1: U$3.GPIO1, X1P0.20.S
- new net ADS_GPIO2: U$3.GPIO2, X1P0.19.S
- new net ADS_PWDN: U$3.PWDN, X1P0.17.S
- new net ADS_START: U$3.START, X1P0.18.S
- new net N$10: C1.2, U$3.PGA1P
- new net N$11: R11.2
- new net N$12: C17.2, U$3.PGA2P
- new net N$17: R3.2, U$3.DOUT
- new net N$18: C17.1, U$3.PGA2N
- new net N$19: R12.2
- new net N$20: C22.2, R10.1, R11.1, R12.1, R8.1
- new net N$21: C22.1, R10.2, U$3.RLDINV
- new net N$22: R8.2, U7.VDD
- new net N$23: C26.1, R16.1, U$3.IN2P
- new net N$24: C25.1, R15.1, U$3.IN2N
- new net N$25: C23.2, R13.1, U$3.IN1N
- new net N$26: C24.2, R14.1, U$3.IN1P
- new net N$27: R13.2, R15.2, U$6.GND
- new net N$28: R16.2, U$6.VDD
- new net N$29: R14.2, U7.GND
- new net N$7: U$3.VCAP1
- new net N$9: C1.1, U$3.PGA1N
- net GND: now also C15.1, C16.1, C18.1, C18.2, C19.1, C19.2, C20.1, C21.1, C23.1, C24.1, C25.2, C26.2, C3.2, C4.1, C5.1, C6.1, U$3.AVSS, U$3.DGND, U$3.VREFN, U$3.VREFP; no longer C1.1, C3.1, C4.2, C5.2, C6.2, U1.GND, U2.GND, U4.GND, U5.GND, U7.GND@18, U7.GND@20
- net MPU_DATA: no longer U7.INT
- net N$1: now also C4.2, U$3.VCAP2; no longer C4.1, U7.REGOUT
- net SCK1: now also U$3.SCLK; no longer U1.SCK, U2.SCK, U4.SCK, U5.SCLK, U7.SCL
- net SDI1: now also U$3.DIN; no longer U1.SDI, U2.SDI, U4.SDI, U5.MOSI, U7.SDA
- net SDO1: now also R3.1; no longer U1.SDO, U2.SDO, U4.SDO, U5.MISO, U7.ADO/SDO
- net VCC: now also C15.2, C16.2, C20.2, C21.2, C5.2, C6.2, U$3.AVDD, U$3.DVDD; no longer C1.2, C3.2, C5.1, U1.VDD, U2.VDD, U4.VDD, U5.VS, U7.RESV1, U7.VDD, U7.VDDIO
Other:
- moved on the sheet: C1, C3, C4, C5, C6

Commit message: revA
Connections:
- removed net MPU_DATA: X1P0.15.S
- new net AGND: C18.1, C18.2, C19.1, C19.2, C20.1, C21.1, C23.1, C24.1, C25.2, C26.2, C3.2, C4.1, U$3.AVSS, U$3.VREFN, U$3.VREFP
- net ADS_CLK: now also X1P0.17.S; no longer U$1P0.25.S
- net ADS_CLKSEL: now also X1P0.20.S; no longer U$1P0.22.S
- net ADS_CS: now also U$3.CS, X1P0.16.S; no longer U$1P0.23.S
- net ADS_DATA: now also X1P0.15.S; no longer U$1P0.21.S
- net ADS_GPIO1: now also U$1P0.21.S; no longer X1P0.20.S
- net ADS_GPIO2: now also U$1P0.23.S; no longer X1P0.19.S
- net ADS_PWDN: now also X1P0.19.S; no longer X1P0.17.S
- net GND: no longer C18.1, C18.2, C19.1, C19.2, C20.1, C21.1, C23.1, C24.1, C25.2, C26.2, C3.2, C4.1, U$3.AVSS, U$3.VREFN, U$3.VREFP
- net N$11: now also U$3.RLDOUT
- net N$19: now also U$3.RLDIN
- net N$7: now also C3.1
- net SWITCH: now also X1P0.14.S; no longer X1P0.16.S
