File: hardware/shield/hrm-shield.brd (EAGLE design)
At the start: 23.9 x 32.2 mm, 37 parts, among them IC3 FM25-DFN, T2 BC846, U1 EM406FLAT, U2 EM406FLAT, U4 EM406FLAT, U5 ADXL362, U6 W25Q16BVZP, U7 MPU-9250, X1 NRF51822-RIGHT

Commit message: scheme with ada1292
Parts:
- removed U1, U2, U4: EM406FLAT, icarus_sensors:EM406-FLAT
- removed U5: ADXL362, icarus_sensors:ADXL362-1:1
- added C15, C18, C19, C20: 1uF, SparkFun-Capacitors:0603-CAP
- added C16, C21: 0.1uF, SparkFun-Capacitors:0603-CAP
- added C17: 4.7nF, SparkFun-Capacitors:0603-CAP
- added C22: 1.5nF, SparkFun-Capacitors:0603-CAP
- added C23, C24, C25, C26: 47pF, SparkFun-Capacitors:0603-CAP
- added R10: 1M, SparkFun-Resistors:0603-RES
- added R11, R3: 0, SparkFun-Resistors:0603-RES
- added R12, R8: 100K, SparkFun-Resistors:0603-RES
- added R13, R14, R15, R16: 51K, SparkFun-Resistors:0603-RES
- added U$3: ADS1292, icarus_sensors:QFN-32-4X4
- added U$6: (no value), icarus_sensors:EM406-2PIN
- C1: value 0.1uF -> 4.7nF
- C3: value 10nF -> 1uF
- C4, C5: value 0.1uF -> 1uF
- U7: value MPU-9250 -> (none); device icarus_sensors:MPU-9250 -> icarus_sensors:EM406-2PIN
- moved U7 72.0 mm to (-1.83, -53.4), flipped to the top
- moved C6 48.1 mm to (-5.89, -17.7), flipped to the top, turned to 0 degrees
- moved C5 45.5 mm to (-5.89, -14.6), flipped to the top, turned to 0 degrees
- moved C3 44.4 mm to (-5.89, -8.53), flipped to the top, turned to 0 degrees
- moved C4 42.9 mm to (-5.89, -11.6), flipped to the top, turned to 0 degrees
- moved C1 40.6 mm to (-5.89, -5.49), flipped to the top, turned to 0 degrees
Connections:
- removed net ADXL_CS: U$1.4, U5.P$8
- removed net ADXL_DATA: U$1.2, U5.P$11
- removed net ADXL_FSYNC: U$1.3, U5.P$9
- removed net BAR1_CS: U$1.6, U1.5
- removed net BAR2_CS: U4.5, X1.2
- removed net BAR3_CS: U2.5, X1.4
- removed net MPU_CS: U7.22, X1.1
- removed net MPU_FSYNC: U7.11, X1.3
- removed net VCCIO: C6.1, U5.P$1
- new net ADS_CLK: U$1.6, U$3.17
- new net ADS_CLKSEL: U$1.3, U$3.14
- new net ADS_CS: U$1.4
- new net ADS_DATA: U$1.2, U$3.22
- new net ADS_GPIO1: U$3.26, X1.2
- new net ADS_GPIO2: U$3.25, X1.4
- new net ADS_PWDN: U$3.15, X1.3
- new net ADS_START: U$3.16, X1.1
- new net N$10: C1.2, U$3.2
- new net N$11: R11.2
- new net N$12: C17.2, U$3.8
- new net N$17: R3.2, U$3.21
- new net N$18: C17.1, U$3.7
- new net N$19: R12.2
- new net N$20: C22.2, R10.1, R11.1, R12.1, R8.1
- new net N$21: C22.1, R10.2, U$3.28
- new net N$22: R8.2, U7.1
- new net N$23: C26.1, R16.1, U$3.6
- new net N$24: C25.1, R15.1, U$3.5
- new net N$25: C23.2, R13.1, U$3.3
- new net N$26: C24.2, R14.1, U$3.4
- new net N$27: R13.2, R15.2, U$6.2
- new net N$28: R16.2, U$6.1
- new net N$29: R14.2, U7.2
- new net N$7: U$3.11
- new net N$9: C1.1, U$3.1
- net GND: now also C15.1, C16.1, C18.1, C18.2, C19.1, C19.2, C20.1, C21.1, C23.1, C24.1, C25.2, C26.2, C3.2, C4.1, C5.1, C6.1, U$3.10, U$3.13, U$3.24, U$3.9; no longer C1.1, C3.1, C4.2, C5.2, C6.2, U1.6, U2.6, U4.6, U5.P$12, U5.P$13, U5.P$16, U7.18, U7.20
- net MPU_DATA: no longer U7.12
- net N$1: now also C4.2, U$3.27; no longer C4.1, U7.10
- net SCK1: now also U$3.20; no longer U1.3, U2.3, U4.3, U5.P$4, U7.23
- net SDI1: now also U$3.19; no longer U1.4, U2.4, U4.4, U5.P$6, U7.24
- net SDO1: now also R3.1; no longer U1.2, U2.2, U4.2, U5.P$7, U7.9
- net VCC: now also C15.2, C16.2, C20.2, C21.2, C5.2, C6.2, U$3.12, U$3.23; no longer C1.2, C3.2, C5.1, U1.1, U2.1, U4.1, U5.P$14, U7.1, U7.13, U7.8
Routing:
- net GND: track 160.4 -> 83.6 mm, vias 4 -> 1
- net VCC: track 118.7 -> 45.7 mm, vias 13 -> 4
- net SDO1: track 58.5 -> 0.00 mm, vias 3 -> 0
- net SCK1: track 55.8 -> 0.00 mm, vias 4 -> 0
- net SDI1: track 42.5 -> 0.00 mm, vias 6 -> 0
- net BAR3_CS: track 22.0 -> 0.00 mm, vias 1 -> 0
- net N$1: track 13.6 -> 0.00 mm, vias 2 -> 0
- net MPU_CS: track 13.0 -> 0.00 mm, vias 1 -> 0
- net BAR2_CS: track 12.1 -> 0.00 mm
- net ADXL_CS: track 12.1 -> 0.00 mm
- net BAR1_CS: track 12.0 -> 0.00 mm, vias 2 -> 0
- net ADXL_FSYNC: track 11.0 -> 0.00 mm
- net MPU_DATA: track 9.91 -> 0.00 mm
- net MPU_FSYNC: track 9.20 -> 0.00 mm
- net ADXL_DATA: track 6.83 -> 0.00 mm
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
Commit message: revA
Parts:
- moved R16 121.9 mm to (18.1, 26.0), turned to 180 degrees
- moved R15 114.3 mm to (15.2, 21.9), turned to 270 degrees
- moved R14 113.0 mm to (7.92, 24.8), turned to 180 degrees
- moved C26 112.0 mm to (18.3, 28.0)
- moved R13 108.5 mm to (13.0, 22.6), turned to 90 degrees
- moved C25 105.2 mm to (13.4, 25.2)
- moved C24 98.4 mm to (8.74, 22.1), turned to 90 degrees
- moved C22 97.5 mm to (2.44, 28.0), turned to 180 degrees
- moved C23 95.7 mm to (10.8, 22.1), turned to 90 degrees
- moved R12 90.4 mm to (2.44, 24.0)
- moved R8 87.4 mm to (2.44, 30.1)
- moved R10 86.4 mm to (2.44, 26.0)
- moved R11 85.3 mm to (2.44, 21.9)
- moved U7 83.9 mm to (6.10, 30.1), turned to 180 degrees
- moved U$6 79.1 mm to (13.0, 30.1), turned to 180 degrees
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Connections:
- removed net MPU_DATA: X1.7
- new net AGND: C18.1, C18.2, C19.1, C19.2, C20.1, C21.1, C23.1, C24.1, C25.2, C26.2, C3.2, C4.1, U$3.10, U$3.13, U$3.9
- net ADS_CLK: now also X1.3; no longer U$1.6
- net ADS_CLKSEL: now also X1.2; no longer U$1.3
- net ADS_CS: now also U$3.18, X1.8; no longer U$1.4
- net ADS_DATA: now also X1.7; no longer U$1.2
- net ADS_GPIO1: now also U$1.2; no longer X1.2
- net ADS_GPIO2: now also U$1.4; no longer X1.4
- net ADS_PWDN: now also X1.4; no longer X1.3
- net GND: no longer C18.1, C18.2, C19.1, C19.2, C20.1, C21.1, C23.1, C24.1, C25.2, C26.2, C3.2, C4.1, U$3.10, U$3.13, U$3.9
- net N$11: now also U$3.30
- net N$19: now also U$3.29
- net N$7: now also C3.1
- net SWITCH: now also X1.10; no longer X1.8
Routing:
- net VCC: track 45.7 -> 116.1 mm, vias 4 -> 6
- net GND: track 83.6 -> 131.8 mm
- net AGND: track 0.00 -> 40.3 mm, vias 0 -> 4
- net N$17: track 0.00 -> 34.3 mm, vias 0 -> 1
- net N$30: track 0.00 -> 25.7 mm
- net N$25: track 0.00 -> 20.7 mm, vias 0 -> 1
- net SCK1: track 0.00 -> 20.2 mm, vias 0 -> 1
- net ADS_CS: track 0.00 -> 20.0 mm
- net SDI1: track 0.00 -> 19.8 mm, vias 0 -> 1
- net ADS_DATA: track 0.00 -> 19.4 mm
- net ADS_PWDN: track 0.00 -> 16.4 mm
- net ADS_CLKSEL: track 0.00 -> 15.8 mm
- net N$23: track 0.00 -> 14.6 mm, vias 0 -> 1
- net N$24: track 0.00 -> 14.2 mm, vias 0 -> 1
- net ADS_CLK: track 0.01 -> 14.2 mm
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- added copper zone on layer 1, net AGND
- added copper zone on layer 16, net AGND
- added copper zone on layer 16, net GND
- added copper zone on layer 16, net N$31

Commit message: revA - fixes
Routing:
- net GND: track 131.8 -> 129.6 mm
Changed lines of the file:
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@@
 <param name="mtCopper" value="0.035mm 0.035mm 0.035mm 0.035mm 0.035mm 0.035mm 0.035mm 0.035mm 0.035mm 0.035mm 0.035mm 0.035mm 0.035mm 0.035mm 0.035mm 0.035mm"/>
 <param name="mtIsolate" value="1.5mm 0.15mm 0.2mm 0.15mm 0.2mm 0.15mm 0.2mm 0.15mm 0.2mm 0.15mm 0.2mm 0.15mm 0.2mm 0.15mm 0.2mm"/>
-<param name="mdWireWire" value="8mil"/>
-<param name="mdWirePad" value="8mil"/>
-<param name="mdWireVia" value="8mil"/>
-<param name="mdPadPad" value="8mil"/>
-<param name="mdPadVia" value="8mil"/>
-<param name="mdViaVia" value="8mil"/>
-<param name="mdSmdPad" value="8mil"/>
-<param name="mdSmdVia" value="8mil"/>
-<param name="mdSmdSmd" value="8mil"/>
+<param name="mdWireWire" value="7mil"/>
+<param name="mdWirePad" value="7mil"/>
+<param name="mdWireVia" value="7mil"/>
+<param name="mdPadPad" value="7mil"/>
+<param name="mdPadVia" value="7mil"/>
+<param name="mdViaVia" value="7mil"/>
+<param name="mdSmdPad" value="7mil"/>
+<param name="mdSmdVia" value="7mil"/>
+<param name="mdSmdSmd" value="7mil"/>
 <param name="mdViaViaSameLayer" value="8mil"/>
 <param name="mnLayersViaInSmd" value="2"/>
@@
 <wire x1="10.899140625" y1="11.076940625" x2="10.99058125" y2="11.076940625" width="0.254" layer="1"/>
 <wire x1="10.99058125" y1="10.988040625" x2="10.99058125" y2="11.076940625" width="0.254" layer="1"/>
-<wire x1="1.4" y1="7.2" x2="2.387159375" y2="6.162040625" width="0.2032" layer="1"/>
-<wire x1="2.387159375" y1="6.162040625" x2="4.55168125" y2="6.162040625" width="0.2032" layer="1"/>
+<wire x1="1.4" y1="7.2" x2="2.082359375" y2="6.238240625" width="0.2032" layer="1"/>
+<wire x1="2.082359375" y1="6.238240625" x2="4.37388125" y2="6.263640625" width="0.2032" layer="1"/>
 <wire x1="10.937240625" y1="11.076940625" x2="10.99058125" y2="11.076940625" width="0.254" layer="1"/>
 <wire x1="10.99058125" y1="11.076940625" x2="9.68248125" y2="9.768840625" width="0.2032" layer="16"/>
@@
 <via x="9.944103125" y="14.645640625" extent="1-16" drill="0.6"/>
 <wire x1="6.55828125" y1="15.98168125" x2="6.568440625" y2="15.971521875" width="0.2032" layer="16"/>
-<wire x1="4.55168125" y1="6.162040625" x2="5.369559375" y2="7.08151875" width="0.2032" layer="1"/>
+<wire x1="4.37388125" y1="6.263640625" x2="5.369559375" y2="7.08151875" width="0.2032" layer="1"/>
 <wire x1="5.369559375" y1="7.08151875" x2="5.369559375" y2="7.785103125" width="0.2032" layer="1"/>
 <wire x1="6.6059" y1="7.619" x2="6.439796875" y2="7.785103125" width="0.2032" layer="16"/>
@@
 <wire x1="13.5772" y1="16.0528" x2="13.5772" y2="14.224" width="0.2032" layer="16"/>
 <wire x1="13.5772" y1="14.224" x2="13.7804" y2="14.0208" width="0.2032" layer="16"/>
-<wire x1="9.22068125" y1="17.198340625" x2="9.827259375" y2="17.198340625" width="0.2032" layer="16"/>
-<wire x1="9.827259375" y1="17.198340625" x2="10.9728" y2="16.0528" width="0.2032" layer="16"/>
 <wire x1="10.9728" y1="16.0528" x2="11.176" y2="16.0528" width="0.2032" layer="16"/>
 <wire x1="11.176" y1="16.0528" x2="11.7856" y2="15.4432" width="0.2032" layer="16"/>
@@
 <contactref element="X1" pad="4"/>
 <wire x1="16.256" y1="21.5392" x2="19.304" y2="21.5392" width="0.2032" layer="16"/>
-<wire x1="19.304" y1="21.5392" x2="21.5392" y2="19.304" width="0.2032" layer="16"/>
-<wire x1="21.5392" y1="19.304" x2="21.5392" y2="16.2608" width="0.2032" layer="16"/>
-<wire x1="21.5392" y1="16.2608" x2="22.6" y2="15.2" width="0.2032" layer="16"/>
+<wire x1="19.304" y1="21.5392" x2="21.6408" y2="19.304" width="0.2032" layer="16"/>
+<wire x1="21.6408" y1="19.304" x2="21.59" y2="16.2608" width="0.2032" layer="16"/>
+<wire x1="21.59" y1="16.2608" x2="22.6" y2="15.2" width="0.2032" layer="16"/>
 </signal>
 <signal name="ADS_START">
@@
 <contactref element="IC3" pad="7"/>
 <contactref element="U$1" pad="15"/>
-<wire x1="4.269740625" y1="4.155440625" x2="2.48158125" y2="4.155440625" width="0.2032" layer="16"/>
-<wire x1="2.48158125" y1="4.155440625" x2="1.526140625" y2="3.2" width="0.2032" layer="16"/>
+<wire x1="4.244340625" y1="4.231640625" x2="2.48158125" y2="4.206240625" width="0.2032" layer="16"/>
+<wire x1="2.48158125" y1="4.206240625" x2="1.526140625" y2="3.2" width="0.2032" layer="16"/>
 <wire x1="1.526140625" y1="3.2" x2="1.4" y2="3.2" width="0.2032" layer="16"/>
-<wire x1="4.269740625" y1="4.155440625" x2="4.38911875" y2="4.27481875" width="0.2032" layer="16"/>
-<wire x1="4.38911875" y1="4.27481875" x2="4.38911875" y2="6.05281875" width="0.2032" layer="16"/>
+<wire x1="4.244340625" y1="4.231640625" x2="4.36371875" y2="4.35101875" width="0.2032" layer="16"/>
+<wire x1="4.36371875" y1="4.35101875" x2="4.38911875" y2="6.05281875" width="0.2032" layer="16"/>
 <wire x1="4.38911875" y1="6.05281875" x2="5.2451" y2="6.9088" width="0.2032" layer="16"/>
 <wire x1="5.2451" y1="6.9088" x2="7.112" y2="6.9088" width="0.2032" layer="16"/>
@@
 <contactref element="C12" pad="1"/>
 <contactref element="U6" pad="2"/>
-<wire x1="1.4" y1="1.2" x2="2.127559375" y2="0.218440625" width="0.2032" layer="16"/>
-<wire x1="2.127559375" y1="0.218440625" x2="4.61518125" y2="0.218440625" width="0.2032" layer="16"/>
-<wire x1="4.61518125" y1="0.218440625" x2="5.38988125" y2="0.891540625" width="0.2032" layer="16"/>
+<wire x1="1.4" y1="1.2" x2="2.127559375" y2="0.193040625" width="0.2032" layer="16"/>
+<wire x1="2.127559375" y1="0.193040625" x2="4.58978125" y2="0.193040625" width="0.2032" layer="16"/>
+<wire x1="4.58978125" y1="0.193040625" x2="5.38988125" y2="0.891540625" width="0.2032" layer="16"/>
 <wire x1="5.38988125" y1="0.891540625" x2="5.38988125" y2="1.64591875" width="0.2032" layer="16"/>
 <wire x1="5.38988125" y1="1.64591875" x2="5.74294375" y2="1.99898125" width="0.2032" layer="16"/>
@@
 <wire x1="12.194540625" y1="8.14578125" x2="11.99388125" y2="8.346440625" width="0.254" layer="16"/>
 <wire x1="12.194540625" y1="6.3754" x2="13.3858" y2="5.184140625" width="0.2032" layer="16"/>
-<wire x1="13.3858" y1="5.184140625" x2="13.4366" y2="4.493259375" width="0.2032" layer="16"/>
-<wire x1="13.4366" y1="4.493259375" x2="12.7762" y2="4.061459375" width="0.2032" layer="16"/>
-<wire x1="12.7762" y1="4.061459375" x2="12.486640625" y2="4.036059375" width="0.2032" layer="16"/>
-<wire x1="12.486640625" y1="4.036059375" x2="12.07008125" y2="3.6195" width="0.2032" layer="16"/>
+<wire x1="13.3858" y1="5.184140625" x2="13.3858" y2="4.4958" width="0.2032" layer="16"/>
+<wire x1="13.3858" y1="4.4958" x2="12.588240625" y2="3.985259375" width="0.2032" layer="16"/>
+<wire x1="12.588240625" y1="3.985259375" x2="12.07008125" y2="3.6195" width="0.2032" layer="16"/>
 <wire x1="12.07008125" y1="3.6195" x2="12.062459375" y2="3.6195" width="0.2032" layer="16"/>
 <wire x1="12.062459375" y1="3.6195" x2="12.04084375" y2="3.597884375" width="0.2032" layer="16"/>
@@
 <signal name="N$30">
 <wire x1="0.2032" y1="18.0848" x2="0.2032" y2="2.4384" width="0.4064" layer="1"/>
-<wire x1="0.2032" y1="2.4384" x2="0.381" y2="2.159" width="0.4064" layer="1"/>
-<wire x1="0.381" y1="2.159" x2="4.2926" y2="2.159" width="0.2032" layer="1"/>
-<wire x1="4.2926" y1="2.159" x2="4.8768" y2="2.2352" width="0.4064" layer="1"/>
+<wire x1="0.2032" y1="2.4384" x2="0.381" y2="2.2352" width="0.4064" layer="1"/>
+<wire x1="0.381" y1="2.2352" x2="4.2926" y2="2.2352" width="0.2032" layer="1"/>
+<wire x1="4.2926" y1="2.2352" x2="4.8768" y2="2.2352" width="0.4064" layer="1"/>
 <wire x1="4.8768" y1="2.2352" x2="5.8928" y2="3.2512" width="0.4064" layer="1"/>
 <wire x1="5.8928" y1="3.2512" x2="8.3312" y2="3.2512" width="0.4064" layer="1"/>
